File: LoRaWAY.kicad_pcb (KiCad board)
At the start: 4 copper layers, 29.8 x 53.6 mm, 59 parts, among them J1 USB4105-GF-A, J2 Sensor connector, J3 ANTENNA, J4 BOOT_SEL, SW1 BOOT, SW2 QRST, SW3 RST, U2 KG200ZABMD, U3 USBLC6-2SC6, U5 AMS1117-3.3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

Commit message: Pre-release v1.0
Parts:
- removed J2: Sensor connector, Connector_JST:JST_EH_S4B-EH_1x04_P2.50mm_Horizontal
- removed U5: AMS1117-3.3, Package_TO_SOT_SMD:SOT-223-3_TabPin2
- added U1: AP7363, LoRaWAY-FTP:TO252-3L_DIO, F.Cu at (158.7, 110.5)
- added kibuzzard-694845CE: G***, kibuzzard-694845CE, F.Cu at (155.6, 90.4)
- added kibuzzard-69502FA5: G***, kibuzzard-69502FA5, F.Cu at (183.2, 79.2)
- C3: value 4u7 -> 22u
- moved J3 18.3 mm to (182.8, 69.6), turned to -90 degrees
- moved C14 14.7 mm to (179.6, 69.2), turned to 90 degrees
- moved R14 12.6 mm to (178.1, 69.7), turned to 0 degrees
- moved C12 11.6 mm to (176.7, 69.2), turned to 90 degrees
- moved C4 5.49 mm to (159.4, 101.2), turned to 0 degrees
- moved C3 4.62 mm to (162.4, 102.0), turned to 90 degrees
- moved TP3 2.88 mm to (183.2, 87.3)
- moved kibuzzard-694845CE 2.77 mm to (155.5, 83.1)
- moved TP4 1.52 mm to (183.2, 89.5)
Connections:
- U2 pad 61: /MODULE_USART2_RTS -> unconnected-(U2A-GPIO1-Pad61)
- U2 pad 62: /MODULE_USART2_CTS -> unconnected-(U2A-GPIO0-Pad62)
- U6 pad 10: /MODULE_USART1_CTS -> unconnected-(U6-MTDI-Pad10)
- U6 pad 9: /MODULE_USART1_RTS -> unconnected-(U6-MTMS-Pad9)
Routing:
- net /BOOT: track 6.92 -> 38.1 mm, vias 0 -> 2
- net /MCU_RST: track 8.09 -> 37.7 mm, vias 1 -> 2
- net /MODUL_UART_TXD: track 1.62 -> 27.4 mm, vias 0 -> 4
- net /ANT_LORA: track 0.00 -> 15.0 mm
- net /SWCLK: track 0.00 -> 12.7 mm
- net /SWDIO: track 0.00 -> 10.9 mm
- net GND: track 49.3 -> 56.2 mm, vias 74 -> 109
- net /MODULE_UART_RXD: track 1.67 -> 7.20 mm
- net /MODULE_RST: track 33.4 -> 37.4 mm
- net /MODULE_USART2_TXD: track 28.7 -> 30.6 mm
- net /MODULE_USART1_CTS: track 1.89 -> 0.00 mm
- net +3V3: track 8.67 -> 9.94 mm, vias 22 -> 30
- net /MODULE_USART2_RXD: track 29.2 -> 30.3 mm
- net /MODULE_USART1_RTS: track 0.77 -> 0.00 mm
- net /VDDSMPS: track 6.54 -> 5.98 mm
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- added copper zone on B.Cu, net GND
Other:
- board size 29.8 x 53.6 mm -> 29.8 x 48 mm

Commit message: Final design
Parts:
- removed kibuzzard-694813BB: G***, kibuzzard-694813BB
- removed kibuzzard-6948142B: G***, kibuzzard-6948142B
- added TP9: TestPoint, TestPoint:TestPoint_Pad_D1.0mm, F.Cu at (157.1, 86.3)
- moved SW2 0.62 mm to (180.4, 102.5)
- moved C9 0.61 mm to (176.7, 101.9)
- moved J3 0.58 mm to (182.2, 69.6)
Routing:
- net Net-(J3-In): track 0.00 -> 2.10 mm
- net +3V3: track 9.94 -> 11.0 mm, vias 30 -> 31
- net /ANT_LORA: track 15.0 -> 15.5 mm
- net /MODULE_RST: track 37.4 -> 38.0 mm
- net GND: track 56.2 -> 56.4 mm, vias 109 -> 366
Other:
- outline, holes or cut-outs redrawn
